Commit message: d1+piper训练配置成功 训练成功

File: source/LeggedManip_Lab/LeggedManip_Lab/assets/d1_piper_l/d1_piper_l.urdf (robot description, URDF)
Before this commit: robot d1_piper_l, 37 links, 36 joints
Joints:
- joint end_effector_joint: origin xyz=0 0 0 rpy=0 0 0 -> xyz=0.0 0 0.10 rpy=0 -1.5707963 0

Commit message: 添加机械臂IK训练配置

File: source/LeggedManip_Lab/LeggedManip_Lab/assets/d1_piper_l/d1_piper_l.urdf (robot description, URDF)
Before this commit: robot d1_piper_l, 37 links, 36 joints
Joints:
- joint end_effector_joint: origin xyz=0.0 0 0.10 rpy=0 -1.5707963 0 -> xyz=0.0 0 0.10 rpy=0 0 0
